File: CAN-SW-STM32L433.kicad_sch (KiCad schematic)
At the start: 37 parts, among them CON12V1 CENTER+, J1 CANBUS, J2 TERM, U1 STM32L433RCT3, U2 MCP2562-E-SN

Commit message: layout and drc complete, fix some silkscreen issues
Parts:
- J1: value CANBUS -> H CAN L
- J2: footprint Connector_PinHeader_1.27mm:PinHeader_1x02_P1.27mm_Vertical -> Connector_PinHeader_2.54mm:PinHeader_1x02_P2.54mm_Vertical
- J3: renamed from UART1; value Conn_01x04 -> UART1
- J4: renamed from SWLINK1; value Conn_ARM_JTAG_SWD_10 -> SWLINK
Changed lines of the file:
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@@
 			)
 		)
-		(property "Value" "CANBUS"
+		(property "Value" "H CAN L"
 			(at 245.11 102.87 0)
 			(effects
@@
 			)
 		)
-		(property "Footprint" "Connector_PinHeader_1.27mm:PinHeader_1x02_P1.27mm_Vertical"
+		(property "Footprint" "Connector_PinHeader_2.54mm:PinHeader_1x02_P2.54mm_Vertical"
 			(at 165.1 22.86 0)
 			(effects
@@
 		(dnp no)
 		(fields_autoplaced yes)
-		(property "Reference" "SWLINK1"
+		(property "Reference" "J4"
 			(at 232.41 67.3099 0)
 			(effects
@@
 			)
 		)
-		(property "Value" "Conn_ARM_JTAG_SWD_10"
+		(property "Value" "SWLINK"
 			(at 232.41 69.8499 0)
 			(effects
@@
 			(project ""
 				(path "/807782eb-8307-4922-8e5a-50da44718f8e"
-					(reference "SWLINK1")
+					(reference "J4")
 					(unit 1)
 				)
@@
 		(dnp no)
 		(fields_autoplaced yes)
-		(property "Reference" "UART1"
+		(property "Reference" "J3"
 			(at 246.38 133.35 0)
 			(effects
@@
 			)
 		)
-		(property "Value" "Conn_01x04"
+		(property "Value" "UART1"
 			(at 246.38 135.89 0)
 			(effects
@@
 					(size 1.27 1.27)
 				)
-				(hide yes)
 			)
 		)
@@
 			(project ""
 				(path "/807782eb-8307-4922-8e5a-50da44718f8e"
-					(reference "UART1")
-					(unit 1)
-				)
+					(reference "J3")
+					(unit 1)
+				)

Commit message: moved power and can connectors, fixed some trace routing
Parts:
- J5: renamed from CON12V1; value CENTER+ -> +12V CENTER +
Changed lines of the file:
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@@
 		(dnp no)
 		(fields_autoplaced yes)
-		(property "Reference" "CON12V1"
+		(property "Reference" "J5"
 			(at 83.82 25.3999 0)
 			(effects
@@
 			)
 		)
-		(property "Value" "CENTER+"
+		(property "Value" "+12V CENTER +"
 			(at 81.28 31.75 0)
 			(effects
@@
 			(project "CAN-SW-STM32L433"
 				(path "/807782eb-8307-4922-8e5a-50da44718f8e"
-					(reference "CON12V1")
+					(reference "J5")
 					(unit 1)
 				)

Commit message: silkscreen tweaks
Parts:
- J1: value H CAN L -> H GND L
- J5: value +12V CENTER + -> CENTER +12V
- renumbered C5V-2 to C5V0
Changed lines of the file:
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@@
 			)
 		)
-		(property "Value" "H CAN L"
+		(property "Value" "H GND L"
 			(at 245.11 102.87 0)
 			(effects
@@
 			)
 		)
-		(property "Value" "+12V CENTER +"
+		(property "Value" "CENTER +12V"
 			(at 81.28 31.75 0)
 			(effects
@@
 		(dnp no)
 		(fields_autoplaced yes)
-		(property "Reference" "C5V-2"
+		(property "Reference" "C5V0"
 			(at 30.48 77.4762 0)
 			(effects
@@
 			(project ""
 				(path "/807782eb-8307-4922-8e5a-50da44718f8e"
-					(reference "C5V-2")
-					(unit 1)
-				)
+					(reference "C5V0")
+					(unit 1)
+				)
